File: syn/syn.kicad_pcb (KiCad board)
At the start: 0 parts

Commit message: up
Parts:
- added BT1: 1.5V, Battery:BatteryHolder_Keystone_2466_1xAAA, F.Cu at (88.5, 52.5)
- added BT2: 1.5V, Battery:BatteryHolder_Keystone_2466_1xAAA, F.Cu at (132.9, 35.3)
- added C1: 100n, Capacitor_SMD:C_2225_5664Metric_Pad1.80x6.60mm_HandSolder, F.Cu at (176.6, 88.4)
- added C2: 10n, Capacitor_SMD:C_2225_5664Metric_Pad1.80x6.60mm_HandSolder, F.Cu at (117.1, 132.8)
- added C3: 100n, Capacitor_SMD:C_2225_5664Metric_Pad1.80x6.60mm_HandSolder, F.Cu at (137.7, 126.0)
- added C4: 22n, Capacitor_SMD:C_2225_5664Metric_Pad1.80x6.60mm_HandSolder, F.Cu at (144.3, 117.5)
- added C5: 22n, Capacitor_SMD:C_2225_5664Metric_Pad1.80x6.60mm_HandSolder, F.Cu at (170.0, 97.4)
- added C6: 1n, Capacitor_SMD:C_2225_5664Metric_Pad1.80x6.60mm_HandSolder, F.Cu at (125.7, 132.8)
- added C7: 1u, Capacitor_SMD:C_2225_5664Metric_Pad1.80x6.60mm_HandSolder, F.Cu at (154.8, 108.4)
- added D1: LED, LED_THT:LED_D3.0mm, F.Cu at (193.1, 78.5)
- added D2: 1N4148, Diode_THT:D_DO-35_SOD27_P7.62mm_Horizontal, F.Cu at (93.2, 121.2)
- added D3: LED, LED_THT:LED_D3.0mm, F.Cu at (186.6, 81.8)
- added D4: LED, LED_THT:LED_D3.0mm, F.Cu at (150.3, 116.2)
- added D5: LED, LED_THT:LED_D3.0mm, F.Cu at (176.0, 95.2)
- added D6: LED, LED_THT:LED_D3.0mm, F.Cu at (143.7, 124.3)
- added D7: LED, LED_THT:LED_D3.0mm, F.Cu at (137.6, 132.9)
- added D8: LED, LED_THT:LED_D3.0mm, F.Cu at (131.7, 132.9)
- added J1: AudioJack2, Connector_Audio:Jack_3.5mm_CUI_SJ1-3535NG_Horizontal, F.Cu at (152.6, 74.3)
- added Q1: BC546, Package_TO_SOT_THT:TO-92_Inline, F.Cu at (161.2, 105.7)
- added Q2: BC546, Package_TO_SOT_THT:TO-92_Inline, F.Cu at (93.7, 134.8)
- added Q3: BC546, Package_TO_SOT_THT:TO-92_Inline, F.Cu at (193.4, 73.2)
- added R1: 1k, Resistor_SMD:R_0815_2038Metric_Pad1.20x4.05mm_HandSolder, F.Cu at (182.6, 98.6)
- added R10: 270k, Resistor_SMD:R_0815_2038Metric_Pad1.20x4.05mm_HandSolder, F.Cu at (193.2, 84.1)
- added R11: 100k, Resistor_SMD:R_0815_2038Metric_Pad1.20x4.05mm_HandSolder, F.Cu at (161.5, 111.0)
- added R12: 100k, Resistor_SMD:R_0815_2038Metric_Pad1.20x4.05mm_HandSolder, F.Cu at (199.7, 78.6)
- added R13: 470, Resistor_SMD:R_0815_2038Metric_Pad1.20x4.05mm_HandSolder, F.Cu at (168.1, 104.3)
- added R14: 470, Resistor_SMD:R_0815_2038Metric_Pad1.20x4.05mm_HandSolder, F.Cu at (160.6, 116.6)
- added R15: 100k, Resistor_SMD:R_0815_2038Metric_Pad1.20x4.05mm_HandSolder, F.Cu at (183.3, 93.0)
- added R16: 100k, Resistor_SMD:R_0815_2038Metric_Pad1.20x4.05mm_HandSolder, F.Cu at (151.0, 121.8)
- added R17: 10K, Resistor_SMD:R_0815_2038Metric_Pad1.20x4.05mm_HandSolder, F.Cu at (144.4, 129.9)
- added R18: 100k, Resistor_SMD:R_0815_2038Metric_Pad1.20x4.05mm_HandSolder, F.Cu at (205.2, 72.8)
- added R19: 100k, Resistor_SMD:R_0815_2038Metric_Pad1.20x4.05mm_HandSolder, F.Cu at (183.3, 87.4)
- added R2: 10k, Resistor_SMD:R_0815_2038Metric_Pad1.20x4.05mm_HandSolder, F.Cu at (200.4, 72.8)
- added R20: 100k, Resistor_SMD:R_0815_2038Metric_Pad1.20x4.05mm_HandSolder, F.Cu at (150.3, 127.4)
- added R21: 10k, Resistor_SMD:R_0815_2038Metric_Pad1.20x4.05mm_HandSolder, F.Cu at (166.3, 111.0)
- added R22: 470, Resistor_SMD:R_0815_2038Metric_Pad1.20x4.05mm_HandSolder, F.Cu at (192.9, 89.7)
- added R23: 470, Resistor_SMD:R_0815_2038Metric_Pad1.20x4.05mm_HandSolder, F.Cu at (172.9, 104.3)
- added R3: 1k, Resistor_SMD:R_0815_2038Metric_Pad1.20x4.05mm_HandSolder, F.Cu at (188.1, 93.0)
- added R4: 100k, Resistor_SMD:R_0815_2038Metric_Pad1.20x4.05mm_HandSolder, F.Cu at (160.6, 122.2)
- added R5: 100k, Resistor_SMD:R_0815_2038Metric_Pad1.20x4.05mm_HandSolder, F.Cu at (165.4, 116.6)
- added R6: 100k, Resistor_SMD:R_0815_2038Metric_Pad1.20x4.05mm_HandSolder, F.Cu at (155.2, 127.4)
- added R7: 10k, Resistor_SMD:R_0815_2038Metric_Pad1.20x4.05mm_HandSolder, F.Cu at (188.1, 87.4)
- added R8: 100k, Resistor_SMD:R_0815_2038Metric_Pad1.20x4.05mm_HandSolder, F.Cu at (156.4, 87.1)
- added R9: 10k, Resistor_SMD:R_0815_2038Metric_Pad1.20x4.05mm_HandSolder, F.Cu at (155.8, 121.8)
- added RV1: 100kB, Potentiometer_THT:Potentiometer_Bourns_PTV09A-1_Single_Vertical, F.Cu at (119.7, 109.7)
- added RV2: 100kB, Potentiometer_THT:Potentiometer_Bourns_PTV09A-1_Single_Vertical, F.Cu at (104.2, 124.1)
- added RV3: 100kB, Potentiometer_THT:Potentiometer_Bourns_PTV09A-1_Single_Vertical, F.Cu at (61.2, 65.1)
- added RV4: 100kB, Potentiometer_THT:Potentiometer_Bourns_PTV09A-1_Single_Vertical, F.Cu at (79.4, 83.8)
- added RV5: 100kB, Potentiometer_THT:Potentiometer_Bourns_PTV09A-1_Single_Vertical, F.Cu at (119.7, 124.1)
- added RV6: 100kB, Potentiometer_THT:Potentiometer_Bourns_PTV09A-1_Single_Vertical, F.Cu at (51.8, 103.1)
- added RV7: 100kA, Potentiometer_THT:Potentiometer_Bourns_PTV09A-1_Single_Vertical, F.Cu at (133.6, 72.6)
- added SW1: Gate1, Button_Switch_THT:SW_PUSH_6mm_H9.5mm, F.Cu at (104.2, 130.8)
- added SW2: Gate2, Button_Switch_THT:SW_PUSH_6mm_H9.5mm, F.Cu at (135.4, 106.4)
- added SW3: Range, Button_Switch_THT:SW_NKK_G1xJP, F.Cu at (161.2, 95.3)
- added SW4: Gate3, Button_Switch_THT:SW_PUSH_6mm_H9.5mm, F.Cu at (93.7, 125.0)
- added SW5: Gate3SW, Button_Switch_THT:SW_NKK_G1xJP, F.Cu at (167.7, 86.3)
- added SW6: Wave, Button_Switch_THT:SW_NKK_G1xJP, F.Cu at (109.1, 80.8)
- added SW7: Mod, Button_Switch_THT:SW_NKK_G1xJP, F.Cu at (161.2, 86.3)
- added SW8: Resonance, Button_Switch_THT:SW_NKK_G1xJP, F.Cu at (135.4, 114.9)
- added SW9: Power, Button_Switch_THT:SW_NKK_G1xJP, F.Cu at (146.0, 106.3)
- added U1: MCP6004, Package_DIP:DIP-14_W7.62mm, F.Cu at (198.4, 114.3)
Other:
- copper layers 0 -> 2
