File: syn/syn.kicad_pcb (KiCad board)
At the start: 2 copper layers, 61 parts, among them J1 AudioJack2, Q1 BC546, Q2 BC546, Q3 BC546, SW1 Gate1, SW2 Gate2, SW3 Range, SW4 Gate3, SW5 Gate3SW, SW6 Wave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

Commit message: up
Parts:
- moved RV1 90.7 mm to (40.8, 64.9)
- moved U1 90.0 mm to (138.1, 47.5), turned to -90 degrees
- moved RV2 48.9 mm to (61.3, 100.6)
- moved SW1 38.3 mm to (81.0, 161.2)
- moved RV6 23.0 mm to (48.6, 125.9)
- moved RV4 18.1 mm to (61.3, 82.3)
Changed lines of the file:
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@@
   (net 53 "unconnected-(SW9-Pad4)")
   (footprint "Potentiometer_THT:Potentiometer_Bourns_PTV09A-1_Single_Vertical" (layer "F.Cu")
-    (at 51.75 103.08)
+    (at 48.65 125.9)
     (descr "Potentiometer, vertical, Bourns PTV09A-1 Single, http://www.bourns.com/docs/Product-Datasheets/ptv09.pdf")
     (tags "Potentiometer vertical Bourns PTV09A-1 Single")
@@
   )
   (footprint "Potentiometer_THT:Potentiometer_Bourns_PTV09A-1_Single_Vertical" (layer "F.Cu")
-    (at 119.65 109.73)
+    (at 40.76 64.93)
     (descr "Potentiometer, vertical, Bourns PTV09A-1 Single, http://www.bourns.com/docs/Product-Datasheets/ptv09.pdf")
     (tags "Potentiometer vertical Bourns PTV09A-1 Single")
@@
     (property "Sheetname" "")
     (attr through_hole)
-    (fp_text reference "BT1" (at 0 -8 180) (layer "F.SilkS")
+    (fp_text reference "BT1" (at 0 -8) (layer "F.SilkS")
       (effects (font (size 1 1) (thickness 0.15)))
     )
@@
   )
   (footprint "Potentiometer_THT:Potentiometer_Bourns_PTV09A-1_Single_Vertical" (layer "F.Cu")
-    (at 79.37 83.76)
+    (at 61.31 82.34)
     (descr "Potentiometer, vertical, Bourns PTV09A-1 Single, http://www.bourns.com/docs/Product-Datasheets/ptv09.pdf")
     (tags "Potentiometer vertical Bourns PTV09A-1 Single")
@@
   )
   (footprint "Potentiometer_THT:Potentiometer_Bourns_PTV09A-1_Single_Vertical" (layer "F.Cu")
-    (at 104.2 124.08)
+    (at 61.31 100.58)
     (descr "Potentiometer, vertical, Bourns PTV09A-1 Single, http://www.bourns.com/docs/Product-Datasheets/ptv09.pdf")
     (tags "Potentiometer vertical Bourns PTV09A-1 Single")
@@
   )
   (footprint "Button_Switch_THT:SW_PUSH_6mm_H9.5mm" (layer "F.Cu")
-    (at 104.25 130.78)
+    (at 81.03 161.24)
     (descr "tactile push button, 6x6mm e.g. PHAP33xx series, height=9.5mm")
     (tags "tact sw push 6mm")
@@
   )
   (footprint "Package_DIP:DIP-14_W7.62mm" (layer "F.Cu")
-    (at 198.36 114.305)
+    (at 138.075 47.5 -90)
     (descr "14-lead though-hole mounted DIP package, row spacing 7.62 mm (300 mils)")
     (tags "THT DIP DIL PDIP 2.54mm 7.62mm 300mil")
@@
     (property "Sheetname" "")
     (attr through_hole)
-    (fp_text reference "U1" (at 3.81 -2.33) (layer "F.SilkS")
-      (effects (font (size 1 1) (thickness 0.15)))
-    )
-    (fp_text value "MCP6004" (at 3.81 17.57) (layer "F.Fab")
-      (effects (font (size 1 1) (thickness 0.15)))
-    )
-    (fp_text user "${REFERENCE}" (at 3.81 7.62) (layer "F.Fab")
+    (fp_text reference "U1" (at 3.81 -2.33 90) (layer "F.SilkS")
+      (effects (font (size 1 1) (thickness 0.15)))
+    )
+    (fp_text value "MCP6004" (at 3.81 17.57 90) (layer "F.Fab")
+      (effects (font (size 1 1) (thickness 0.15)))
+    )
+    (fp_text user "${REFERENCE}" (at 3.81 7.62 90) (layer "F.Fab")
       (effects (font (size 1 1) (thickness 0.15)))
     )
@@
     (fp_line (start 6.985 -1.27) (end 6.985 16.51) (layer "F.Fab") (width 0.1))
     (fp_line (start 0.635 -0.27) (end 1.635 -1.27) (layer "F.Fab") (width 0.1))
-    (pad "1" thru_hole rect locked (at 0 0) (size 1.6 1.6) (drill 0.8) (layers *.Cu *.Mask)
+    (pad "1" thru_hole rect locked (at 0 0 270) (size 1.6 1.6) (drill 0.8) (layers *.Cu *.Mask)
       (net 38 "TRI_SAW") (pintype "output"))
-    (pad "2" thru_hole oval locked (at 0 2.54) (size 1.6 1.6) (drill 0.8) (layers *.Cu *.Mask)
+    (pad "2" thru_hole oval locked (at 0 2.54 270) (size 1.6 1.6) (drill 0.8) (layers *.Cu *.Mask)
       (net 5 "Net-(C2-Pad1)") (pinfunction "-") (pintype "input"))
-    (pad "3" thru_hole oval locked (at 0 5.08) (size 1.6 1.6) (drill 0.8) (layers *.Cu *.Mask)
+    (pad "3" thru_hole oval locked (at 0 5.08 270) (size 1.6 1.6) (drill 0.8) (layers *.Cu *.Mask)
       (net 2 "GND") (pinfunction "+") (pintype "input"))
-    (pad "4" thru_hole oval locked (at 0 7.62) (size 1.6 1.6) (drill 0.8) (layers *.Cu *.Mask)
+    (pad "4" thru_hole oval locked (at 0 7.62 270) (size 1.6 1.6) (drill 0.8) (layers *.Cu *.Mask)
       (net 20 "VCC") (pinfunction "V+") (pintype "power_in"))
-    (pad "5" thru_hole oval locked (at 0 10.16) (size 1.6 1.6) (drill 0.8) (layers *.Cu *.Mask)
+    (pad "5" thru_hole oval locked (at 0 10.16 270) (size 1.6 1.6) (drill 0.8) (layers *.Cu *.Mask)
       (net 39 "Net-(R10-Pad1)") (pinfunction "+") (pintype "input"))
-    (pad "6" thru_hole oval locked (at 0 12.7) (size 1.6 1.6) (drill 0.8) (layers *.Cu *.Mask)
+    (pad "6" thru_hole oval locked (at 0 12.7 270) (size 1.6 1.6) (drill 0.8) (layers *.Cu *.Mask)
       (net 2 "GND") (pinfunction "-") (pintype "input"))
-    (pad "7" thru_hole oval locked (at 0 15.24) (size 1.6 1.6) (drill 0.8) (layers *.Cu *.Mask)
+    (pad "7" thru_hole oval locked (at 0 15.24 270) (size 1.6 1.6) (drill 0.8) (layers *.Cu *.Mask)
       (net 42 "Net-(R10-Pad2)") (pintype "output"))
-    (pad "8" thru_hole oval locked (at 7.62 15.24) (size 1.6 1.6) (drill 0.8) (layers *.Cu *.Mask)
+    (pad "8" thru_hole oval locked (at 7.62 15.24 270) (size 1.6 1.6) (drill 0.8) (layers *.Cu *.Mask)
       (net 13 "Net-(D1-Pad1)") (pintype "output"))
-    (pad "9" thru_hole oval locked (at 7.62 12.7) (size 1.6 1.6) (drill 0.8) (layers *.Cu *.Mask)
+    (pad "9" thru_hole oval locked (at 7.62 12.7 270) (size 1.6 1.6) (drill 0.8) (layers *.Cu *.Mask)
       (net 4 "Net-(C1-Pad2)") (pinfunction "-") (pintype "input"))
-    (pad "10" thru_hole oval locked (at 7.62 10.16) (size 1.6 1.6) (drill 0.8) (layers *.Cu *.Mask)
+    (pad "10" thru_hole oval locked (at 7.62 10.16 270) (size 1.6 1.6) (drill 0.8) (layers *.Cu *.Mask)
       (net 35 "Net-(R5-Pad2)") (pinfunction "+") (pintype "input"))
-    (pad "11" thru_hole oval locked (at 7.62 7.62) (size 1.6 1.6) (drill 0.8) (layers *.Cu *.Mask)
+    (pad "11" thru_hole oval locked (at 7.62 7.62 270) (size 1.6 1.6) (drill 0.8) (layers *.Cu *.Mask)
       (net 22 "VSS") (pinfunction "V-") (pintype "power_in"))
-    (pad "12" thru_hole oval locked (at 7.62 5.08) (size 1.6 1.6) (drill 0.8) (layers *.Cu *.Mask)
+    (pad "12" thru_hole oval locked (at 7.62 5.08 270) (size 1.6 1.6) (drill 0.8) (layers *.Cu *.Mask)
       (net 2 "GND") (pinfunction "+") (pintype "input"))
-    (pad "13" thru_hole oval locked (at 7.62 2.54) (size 1.6 1.6) (drill 0.8) (layers *.Cu *.Mask)
+    (pad "13" thru_hole oval locked (at 7.62 2.54 270) (size 1.6 1.6) (drill 0.8) (layers *.Cu *.Mask)
       (net 8 "Net-(C4-Pad1)") (pinfunction "-") (pintype "input"))
-    (pad "14" thru_hole oval locked (at 7.62 0) (size 1.6 1.6) (drill 0.8) (layers *.Cu *.Mask)
+    (pad "14" thru_hole oval locked (at 7.62 0 270) (size 1.6 1.6) (drill 0.8) (layers *.Cu *.Mask)
       (net 10 "Net-(C5-Pad2)") (pintype "output"))
     (model "${KICAD6_3DMODEL_DIR}/Package_DIP.3dshapes/DIP-14_W7.62mm.wrl"

Commit message: up
Parts:
- removed D8: LED, LED_THT:LED_D3.0mm
- removed Q3: BC546, Package_TO_SOT_THT:TO-92_Inline
- removed R23: 470, Resistor_SMD:R_0815_2038Metric_Pad1.20x4.05mm_HandSolder
- added Q4: BC846, Package_TO_SOT_SMD:SOT-23, F.Cu at (81.4, 29.5)
- BT1, BT2: moved to B.Cu
- C1, C2, C3, C4, C5, C6, C7: footprint Capacitor_SMD:C_2225_5664Metric_Pad1.80x6.60mm_HandSolder -> Capacitor_SMD:C_0805_2012Metric_Pad1.18x1.45mm_HandSolder
- J1: value AudioJack2 -> 35RAPC2BV4; footprint Connector_Audio:Jack_3.5mm_CUI_SJ1-3535NG_Horizontal -> 35RAPC2BV4:SWITCHCRAFT_35RAPC2BV4
- Q1, Q2: value BC546 -> BC846; footprint Package_TO_SOT_THT:TO-92_Inline -> Package_TO_SOT_SMD:SOT-23
- R1, R10, R11, R12, R13, R14, R15, R16, R17, R18, R19, R2, R20, R21, R22, R3, R4, R5, R6, R7, R8, R9: footprint Resistor_SMD:R_0815_2038Metric_Pad1.20x4.05mm_HandSolder -> Resistor_SMD:R_0805_2012Metric_Pad1.20x1.40mm_HandSolder
- moved R2 164.3 mm to (52.0, 143.2), turned to -90 degrees
- moved R12 157.4 mm to (45.9, 45.5)
- moved D1 151.5 mm to (56.2, 143.2)
- moved R3 146.1 mm to (52.8, 37.9)
- moved R10 143.3 mm to (55.2, 45.6)
- moved R18 132.6 mm to (76.8, 39.8), turned to 180 degrees
- moved R5 132.5 mm to (50.5, 50.8)
- moved R7 130.7 mm to (70.0, 143.3), turned to -90 degrees
- moved R11 128.8 mm to (50.6, 45.6), turned to 180 degrees
- moved R14 128.4 mm to (57.4, 40.2)
- moved D3 128.2 mm to (74.1, 143.2)
- moved R6 126.1 mm to (54.9, 50.8)
- moved R21 122.1 mm to (75.3, 29.7)
- moved R1 118.5 mm to (76.8, 45.4), turned to 180 degrees
- moved R15 115.1 mm to (81.2, 39.8), turned to 180 degrees
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Connections:
- Q1 pad 1: Net-(D5-Pad1) -> Net-(D1-Pad1)
- Q1 pad 2: Net-(D1-Pad1) -> Net-(Q1-Pad2)
- Q1 pad 3: Net-(Q1-Pad3) -> Net-(D5-Pad1)
- Q2 pad 1: Net-(D6-Pad1) -> Net-(Q2-Pad1)
- Q2 pad 3: Net-(Q2-Pad3) -> Net-(D6-Pad1)
- R13 pad 1: Net-(Q1-Pad3) -> Net-(Q1-Pad2)
- R14 pad 1: Net-(Q2-Pad3) -> Net-(Q2-Pad2)
- RV7 pad 2: Net-(J1-PadT) -> Net-(J1-Pad2)
- SW6 pad 3: unconnected-(SW6-Pad3) -> (no net)
- SW6 pad 5: Net-(Q2-Pad2) -> Net-(Q2-Pad1)
- SW7 pad 5: Net-(Q2-Pad2) -> Net-(Q2-Pad1)
- SW9 pad 1: unconnected-(SW9-Pad1) -> (no net)
- SW9 pad 4: unconnected-(SW9-Pad4) -> (no net)
Routing:
- net Net-(D1-Pad1): track 0.00 -> 179.0 mm, vias 0 -> 8
- net Net-(C1-Pad2): track 0.00 -> 168.3 mm, vias 0 -> 1
- net VSS: track 0.00 -> 167.9 mm, vias 0 -> 4
- net VCC: track 0.00 -> 130.7 mm, vias 0 -> 6
- net Net-(R21-Pad1): track 0.00 -> 130.1 mm, vias 0 -> 2
- net Net-(Q2-Pad2): track 0.00 -> 115.6 mm, vias 0 -> 4
- net TRI_SAW: track 0.00 -> 95.9 mm, vias 0 -> 2
- net Net-(R10-Pad2): track 0.00 -> 85.0 mm, vias 0 -> 2
- net Net-(C2-Pad1): track 0.00 -> 84.0 mm, vias 0 -> 2
- net Net-(C5-Pad2): track 0.00 -> 81.7 mm, vias 0 -> 4
- net Net-(C4-Pad1): track 0.00 -> 81.4 mm, vias 0 -> 2
- net Net-(R15-Pad2): track 0.00 -> 75.0 mm, vias 0 -> 6
- net Net-(R1-Pad1): track 0.00 -> 68.0 mm, vias 0 -> 2
- net Net-(D7-Pad2): track 0.00 -> 67.1 mm, vias 0 -> 2
- net Net-(Q1-Pad2): track 0.00 -> 66.7 mm, vias 0 -> 6
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- added copper zone on B.Cu, net GND
- added copper zone on F.Cu, net GND
Other:
- board outline added: 83.9 x 145.5 mm
