File: syn/syn.kicad_sch (KiCad schematic)
At the start: 49 parts

Commit message: init
Parts:
- gave numbers to parts that had none: 45
Connections:
- net at C6.1: now also SW6.1 (A)
- no-connect marks 2 -> 5

Commit message: fix
Parts:
- removed SW2: SW_Push_SPDT, symbol Switch:SW_Push_SPDT
- added C?: 100n, symbol Device:C
- added SW?: Range, symbol Switch:SW_Push_DPDT
- added U?: MCP6004, symbol Amplifier_Operational:MCP6004
- SW1: value SW_Push_DPDT -> Range
- SW3, SW4: value SW_Push_DPDT -> Wave
- SW5: value SW_Push_DPDT -> Mod
Connections:
- net at C3.1, R5.2, R6.2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: now also C?.1
- net at R8.1, SW4.4 (A), U1.8: now also SW?.3 (C), SW?.5 (B); no longer C3.2
- net at SW4.6 (C): now also SW?.2 (B)
- net at R12.2, R14.2: now also SW?.1 (A)
- new net: C3.2, SW?.4 (A)
- new net: C?.2, SW?.6 (C)

Commit message: structure
Parts:
- removed C3, C?: 100n, symbol Device:C
- removed D2: 1N4148, Diode_THT:D_DO-35_SOD27_P7.62mm_Horizontal, symbol Diode:1N4148
- removed R10: 270k, symbol Device:R
- removed R12, R8: 100k, symbol Device:R
- removed SW4: Wave, symbol Switch:SW_Push_DPDT
- removed SW6: SW_Push_SPDT, symbol Switch:SW_Push_SPDT
- removed SW?: Range, symbol Switch:SW_Push_DPDT
- removed U1: TL074, symbol Amplifier_Operational:TL074
- removed U2: LM741, symbol Amplifier_Operational:LM741
- removed U?: MCP6004, symbol Amplifier_Operational:MCP6004
- added BT1, BT2: 1.5V, Battery:BatteryHolder_Keystone_2466_1xAAA, symbol Device:Battery_Cell
- added C1: 100n, symbol Device:C
- added D1, D3, D4, D5, D6, D7: LED, symbol Device:LED
- added Q1, Q2: BC546, Package_TO_SOT_THT:TO-92_Inline, symbol Transistor_BJT:BC546
- added R13, R22: 470, symbol Device:R
- added R7, R9: 10k, symbol Device:R
- added RV3, RV4: 100kB, symbol Device:R_Potentiometer
- added SW1, SW2, SW4: SW_Push, symbol Switch:SW_Push
- added SW5: SW_SPST, symbol Switch:SW_SPST
- added SW8: Resonance, symbol Switch:SW_SPST
- added SW9: Power, symbol Switch:SW_Push_DPDT
- added U1: MCP6004, symbol Amplifier_Operational:MCP6004
- R14: value 100k -> 470
- R17: value 100k -> 10K
- R2: value 1k -> 10k
- R5: value 1k -> 100k
- RV7: renamed from RV4; value 100k -> 100kA
- renumbered C1 to C2, C2 to C3, D1 to D2, Q1 to Q3, R9 to R10, R13 to R12, R16 to R15, R15 to R16, R7 to R8, RV3 to RV5, RV5 to RV6, SW1 to SW3, SW3 to SW6, SW5 to SW7
Connections:
- net GND: now also R14.2, R5.1, BT1.2 (-), BT2.1 (+), C1.1, R13.2, U1.12 (+), U1.3 (+), U1.6 (-); no longer R14.1, R2.2
- net at C2.1, C3.1, R3.2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: now also U1.2 (-)
- net TRI_SAW: now reaches R8.1, SW3.3 (C), SW3.5 (B), SW6.4 (A)
- net TRI_SAW: now also U1.1
- net at R5.2: now also R6.1, U1.10 (+); no longer R6.2
- net at C6.1: now also SW8.2 (B)
- net at C5.2, C6.2, C7.1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: now also U1.14
- net at RV2.1: now also RV2.2, C1.2, RV3.1, RV3.2, RV4.1, RV4.2, U1.9 (-)
- net at C4.1, R17.2, R18.2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: now also SW8.1 (A), U1.13 (-)
- net at R10.1, R8.2: now also U1.5 (+)
- net at R10.2, R11.1, RV1.1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: now also U1.7
- net at R15.1: now also R6.2, D1.1 (K), D3.1 (K), D4.1 (K), Q1.2 (B), U1.8
- net at SW6.5 (B), SW7.5 (B): now also Q2.2 (B)
- net SEC_WAVE: now reaches SW3.2 (B), SW6.6 (C)
- net SQR: now reaches R11.2, R12.2, SW3.1 (A)
- net at C4.2, C5.1, Q3.3 (E): now also R19.2; no longer R19.1
- net at Q3.1 (C): now also R19.1; no longer R19.2
- net +9V renamed VCC
- net VCC: now also D5.2 (A), D6.2 (A), R22.1, SW9.3 (C), U1.4 (V+)
- net -9V renamed VSS
- net VSS: now also D7.1 (K), SW9.6 (C), U1.11 (V-)
- new net: D5.1 (K), Q1.1 (C)
- new net: Q1.3 (E), R13.1
- new net: D4.2 (A), SW4.1, SW5.2 (B)
- new net: R9.2, SW4.2, SW5.1 (A)
- new net: D7.2 (A), R22.2
- new net: D1.2 (A), SW1.1
- new net: R2.2, SW1.2
- new net: D6.1 (K), Q2.1 (C)
- new net: BT1.1 (+), SW9.2 (B)
- new net: BT2.2 (-), SW9.5 (B)
- new net: R9.1, RV4.3
- new net: D3.2 (A), SW2.1
- new net: R7.1, RV3.3
- new net: R7.2, SW2.2
- new net: Q2.3 (E), R14.1
- no-connect marks 5 -> 3
Other:
- note added: "2 x AAA"
- note added: "Audio 10n Cap (450 - 1 Hz) LFO 100n Cap (50 - 0.08 Hz)"
- note added: "Closed = Low Reso."
- note added: "Cutoff"
- note added: "Freq"
- note added: "Gates"
- note added: "OSC 1"
- note added: "OSC 1 / 2 Balance"
- note added: "OSC 2"
- note added: "Output"
- note added: "Power"
- note added: "Range"
- note added: "Resonance"
- note added: "Route"
- note added: "VCF LP"
- note added: "square"
- note added: "tri saw"
- note added: "tri/saw or tri/sqr"
- note added: "tri/saw/sqr"
- moved on the sheet: C4, C5, C7, J1, Q3, R15, R18, R19, R21, R8, RV5, RV6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

Commit message: structure
Parts:
- added D8: LED, symbol Device:LED
- added R23: 470, symbol Device:R
Connections:
- net VCC: now also R23.1
- net VSS: now also D8.1 (K)
- new net: D8.2 (A), R23.2
Other:
- moved on the sheet: BT1, BT2, D7, J1, R17, R22, RV7, SW9, U1E

Commit message: up
Parts:
- C1, C2, C3, C4, C5, C6, C7: footprint (none) -> Capacitor_SMD:C_2225_5664Metric_Pad1.80x6.60mm_HandSolder
- D1, D3, D4, D5, D6, D7, D8: footprint (none) -> LED_THT:LED_D3.0mm
- J1: footprint (none) -> Connector_Audio:Jack_3.5mm_CUI_SJ1-3535NG_Horizontal
- R1, R10, R11, R12, R13, R14, R15, R16, R17, R18, R19, R2, R20, R21, R22, R23, R3, R4, R5, R6, R7, R8, R9: footprint (none) -> Resistor_SMD:R_0815_2038Metric_Pad1.20x4.05mm_HandSolder
- RV1, RV2, RV3, RV4, RV5, RV6, RV7: footprint (none) -> Potentiometer_THT:Potentiometer_Bourns_PTV09A-1_Single_Vertical
- SW1: value SW_Push -> Gate1; footprint (none) -> Button_Switch_THT:SW_PUSH_6mm_H9.5mm
- SW2: value SW_Push -> Gate2; footprint (none) -> Button_Switch_THT:SW_PUSH_6mm_H9.5mm
- SW3, SW6, SW7, SW8, SW9: footprint (none) -> Button_Switch_THT:SW_NKK_G1xJP
- SW4: value SW_Push -> Gate3; footprint (none) -> Button_Switch_THT:SW_PUSH_6mm_H9.5mm
- SW5: value SW_SPST -> Gate3SW; footprint (none) -> Button_Switch_THT:SW_NKK_G1xJP
- U1: footprint (none) -> Package_DIP:DIP-14_W7.62mm

Commit message: up
Parts:
- J1: footprint Connector_Audio:Jack_3.5mm_CUI_SJ1-3535NG_Horizontal -> (none)
Changed lines of the file:
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@@
       (effects (font (size 1.27 1.27)) (justify right))
     )
-    (property "Footprint" "Connector_Audio:Jack_3.5mm_CUI_SJ1-3535NG_Horizontal" (id 2) (at 275.844 107.442 0)
+    (property "Footprint" "" (id 2) (at 275.844 107.442 0)
       (effects (font (size 1.27 1.27)) hide)
     )
@@
     )
     (path "/b5089c97-a564-4bf6-b741-fac03e0240fa"
-      (reference "J1") (unit 1) (value "AudioJack2") (footprint "Connector_Audio:Jack_3.5mm_CUI_SJ1-3535NG_Horizontal")
+      (reference "J1") (unit 1) (value "AudioJack2") (footprint "")
     )
     (path "/0d687931-25dd-4c0c-996a-978c8b96e021"

Commit message: up
Parts:
- removed D8: LED, LED_THT:LED_D3.0mm, symbol Device:LED
- removed J1: AudioJack2, symbol Connector:AudioJack2
- removed Q1, Q2, Q3: BC546, Package_TO_SOT_THT:TO-92_Inline, symbol Transistor_BJT:BC546
- removed R23: 470, Resistor_SMD:R_0815_2038Metric_Pad1.20x4.05mm_HandSolder, symbol Device:R
- added J1: 35RAPC2BV4, 35RAPC2BV4:SWITCHCRAFT_35RAPC2BV4, symbol 35RAPC2BV4:35RAPC2BV4
- added Q1, Q2, Q4: BC846, Package_TO_SOT_SMD:SOT-23, symbol Transistor_BJT:BC846
- C1, C2, C3, C4, C5, C6, C7: footprint Capacitor_SMD:C_2225_5664Metric_Pad1.80x6.60mm_HandSolder -> Capacitor_SMD:C_0805_2012Metric_Pad1.18x1.45mm_HandSolder
- R1, R10, R11, R12, R13, R14, R15, R16, R17, R18, R19, R2, R20, R21, R22, R3, R4, R5, R6, R7, R8, R9: footprint Resistor_SMD:R_0815_2038Metric_Pad1.20x4.05mm_HandSolder -> Resistor_SMD:R_0805_2012Metric_Pad1.20x1.40mm_HandSolder
Connections:
- net GND: now also J1.1
- net at D5.1 (K): now also Q1.3 (C)
- net at D1.1 (K), D3.1 (K), D4.1 (K)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: now also Q1.1 (B)
- net at R13.1: now also Q1.2 (E)
- net at D6.1 (K): now also Q2.3 (C)
- net at R21.2: now also Q4.1 (B)
- net at RV7.2: now also J1.2
- net at SW6.5 (B), SW7.5 (B): now also Q2.1 (B)
- net at C4.2, C5.1, R19.2: now also Q4.2 (E)
- net at R19.1: now also Q4.3 (C)
- net at R14.1: now also Q2.2 (E)
Other:
- moved on the sheet: RV7
